File: LEDsupply.sch (KiCad schematic (older format))
At the start: 16 parts, among them U1 MIC2954, U2 MCP4018-502

Commit message: Added a KK series connector
Parts:
- JP3: value Conn_01x03_Female -> KK_3way; footprint Connector_PinHeader_2.54mm:PinHeader_1x03_P2.54mm_Vertical -> Connector_Molex:Molex_KK-254_AE-6410-03A_1x03_P2.54mm_Vertical; Manufacturer (none) -> Molex; Note (none) -> KK 254 Wire-to-Board Header; Order Code (none) -> 9731156; Package (none) -> 2.54mm; Part Number (none) -> 22-27-2031; Supplier (none) -> Farnell
Connections:
- net GND: now also JP3.1 (Pin_1); no longer JP3.3 (Pin_3)
- net VREGOUT: now also JP3.3 (Pin_3); no longer JP3.1 (Pin_1)
Changed lines of the file:
@@
-	1    0    0    -1
-$EndComp
-$Comp
-L Connector:Conn_01x03_Female JP3
-U 1 1 5FB13D6B
-P 7700 2100
-F 0 "JP3" H 7728 2126 50  0000 L CNN
-F 1 "Conn_01x03_Female" H 7728 2035 50  0000 L CNN
-F 2 "Connector_PinHeader_2.54mm:PinHeader_1x03_P2.54mm_Vertical" H 7700 2100 50  0001 C CNN
-F 3 "~" H 7700 2100 50  0001 C CNN
-	1    7700 2100
 	1    0    0    -1
 $EndComp
@@
 	1    0    0    -1
 $EndComp
+$Comp
+L Connector:Conn_01x03_Female JP3
+U 1 1 5FB13D6B
+P 7700 2100
+F 0 "JP3" H 7728 2126 50  0000 L CNN
+F 1 "KK_3way" H 7728 2035 50  0000 L CNN
+F 2 "Connector_Molex:Molex_KK-254_AE-6410-03A_1x03_P2.54mm_Vertical" H 7700 2100 50  0001 C CNN
+F 3 "~" H 7700 2100 50  0001 C CNN
+F 4 "22-27-2031" H 7700 2100 50  0001 C CNN "Part Number"
+F 5 "Molex" H 7700 2100 50  0001 C CNN "Manufacturer"
+F 6 "2.54mm" H 7700 2100 50  0001 C CNN "Package"
+F 7 "Farnell" H 7700 2100 50  0001 C CNN "Supplier"
+F 8 "9731156" H 7700 2100 50  0001 C CNN "Order Code"
+F 9 "KK 254 Wire-to-Board Header" H 7700 2100 50  0001 C CNN "Note"
+	1    7700 2100
+	1    0    0    1
+$EndComp
 $EndSCHEMATC

Commit message: Added I2C pullup resistors, fixed H1 label position, changed R4 from 20 to 24k
Parts:
- added R1, R2: 2k2, Resistor_SMD:R_0603_1608Metric, symbol Device:R
- R4: renamed from R2; value 20k -> 24k
- renumbered JP2 to JP1, JP1 to JP2, R1 to R3, R3 to R5, R4 to R6, R5 to R7
Connections:
- net +5V: now also R1.1, R2.1
- net SCL: now also R1.2
- net SDA: now also R2.2
Other:
- moved on the sheet: JP1
Changed lines of the file:
@@
 	5350 2600 4800 2600
 $Comp
-L Device:R R4
+L Device:R R6
 U 1 1 5FAE1ED0
 P 5850 2300
-F 0 "R4" H 5920 2346 50  0000 L CNN
+F 0 "R6" H 5920 2346 50  0000 L CNN
 F 1 "360k" H 5920 2255 50  0000 L CNN
 F 2 "Resistor_SMD:R_0603_1608Metric" V 5780 2300 50  0001 C CNN
@@
 Connection ~ 5350 2000
 $Comp
-L Device:R R3
+L Device:R R5
 U 1 1 5FAE331A
 P 5350 2850
-F 0 "R3" H 5420 2896 50  0000 L CNN
+F 0 "R5" H 5420 2896 50  0000 L CNN
 F 1 "20k" H 5420 2805 50  0000 L CNN
 F 2 "Resistor_SMD:R_0603_1608Metric" V 5280 2850 50  0001 C CNN
@@
 19.0V - 23.5V\n21.0V (default)
 $Comp
-L Connector:Mini-DIN-6 JP2
+L Connector:Mini-DIN-6 JP1
 U 1 1 5FAF9EF5
-P 2500 4400
-F 0 "JP2" H 2500 4767 50  0000 C CNN
-F 1 "Mini-DIN-6" H 2500 4676 50  0000 C CNN
-F 2 "jakub:MiniDIN6way" H 2500 4400 50  0001 C CNN
-F 3 "http://service.powerdynamics.com/ec/Catalog17/Section%2011.pdf" H 2500 4400 50  0001 C CNN
-F 4 "PSG01567" H 2500 4400 50  0001 C CNN "Part Number"
-F 5 "Pro Signal" H 2500 4400 50  0001 C CNN "Manufacturer"
-F 6 "Chassis" H 2500 4400 50  0001 C CNN "Package"
-F 7 "Farnell" H 2500 4400 50  0001 C CNN "Supplier"
-F 8 "1280671" H 2500 4400 50  0001 C CNN "Order Code"
-F 9 "6way mini DIN Connector" H 2500 4400 50  0001 C CNN "Note"
-	1    2500 4400
-	1    0    0    -1
-$EndComp
-Wire Wire Line
-	2800 4300 3900 4300
-Wire Wire Line
-	2800 4500 3050 4500
+P 2000 4400
+F 0 "JP1" H 2000 4767 50  0000 C CNN
+F 1 "Mini-DIN-6" H 2000 4676 50  0000 C CNN
+F 2 "jakub:MiniDIN6way" H 2000 4400 50  0001 C CNN
+F 3 "http://service.powerdynamics.com/ec/Catalog17/Section%2011.pdf" H 2000 4400 50  0001 C CNN
+F 4 "PSG01567" H 2000 4400 50  0001 C CNN "Part Number"
+F 5 "Pro Signal" H 2000 4400 50  0001 C CNN "Manufacturer"
+F 6 "Chassis" H 2000 4400 50  0001 C CNN "Package"
+F 7 "Farnell" H 2000 4400 50  0001 C CNN "Supplier"
+F 8 "1280671" H 2000 4400 50  0001 C CNN "Order Code"
+F 9 "6way mini DIN Connector" H 2000 4400 50  0001 C CNN "Note"
+	1    2000 4400
+	1    0    0    -1
+$EndComp
+Wire Wire Line
+	2300 4300 2750 4300
+Wire Wire Line
+	2300 4500 3050 4500
 Wire Wire Line
 	3050 4500 3050 4400
@@
 	3050 4400 3900 4400
 Wire Wire Line
-	2800 4400 2900 4400
-Wire Wire Line
-	2900 4400 2900 4700
+	2300 4400 2400 4400
+Wire Wire Line
+	2400 4400 2400 4700
 Wire Wire Line
 	3500 4200 3500 4750
 $Comp
-L power:GND #PWR02
+L power:GND #PWR01
 U 1 1 5FAFE96F
-P 2900 4700
-F 0 "#PWR02" H 2900 4450 50  0001 C CNN
-F 1 "GND" H 2905 4527 50  0000 C CNN
-F 2 "" H 2900 4700 50  0001 C CNN
-F 3 "" H 2900 4700 50  0001 C CNN
-	1    2900 4700
-	1    0    0    -1
-$EndComp
-Wire Wire Line
-	2200 4400 2100 4400
-Wire Wire Line
-	2100 4400 2100 3800
-Wire Wire Line
-	2100 3800 3500 3800
+P 2400 4700
+F 0 "#PWR01" H 2400 4450 50  0001 C CNN
+F 1 "GND" H 2405 4527 50  0000 C CNN
+F 2 "" H 2400 4700 50  0001 C CNN
+F 3 "" H 2400 4700 50  0001 C CNN
+	1    2400 4700
+	1    0    0    -1
+$EndComp
+Wire Wire Line
+	1700 4400 1600 4400
+Wire Wire Line
+	1600 4400 1600 3800
+Wire Wire Line
+	1600 3800 2750 3800
 $Comp
 L Potentiometer_Digital:MCP4018-xxxxLT U2
@@
 $EndComp
 NoConn ~ 4700 4100
-Text Notes 2300 5150 0    50   ~ 0
+Text Notes 1800 5150 0    50   ~ 0
 cable 3400059
 Wire Wire Line
 	2700 2000 3150 2000
 $Comp
-L Connector:Barrel_Jack_Switch_Pin3Ring JP1
+L Connector:Barrel_Jack_Switch_Pin3Ring JP2
 U 1 1 5FB11308
 P 2400 2100
-F 0 "JP1" H 2457 2417 50  0000 C CNN
+F 0 "JP2" H 2457 2417 50  0000 C CNN
 F 1 "Barrel_Jack_Switch_Pin3Ring" H 2457 2326 50  0000 C CNN
 F 2 "jakub:2.1mmBarrelJackTop" H 2450 2060 50  0001 C CNN
@@
 	2800 2200 2800 2300
 $Comp
-L power:GND #PWR01
+L power:GND #PWR02
 U 1 1 5FB1347D
 P 2800 2300
-F 0 "#PWR01" H 2800 2050 50  0001 C CNN
+F 0 "#PWR02" H 2800 2050 50  0001 C CNN
 F 1 "GND" H 2805 2127 50  0000 C CNN
 F 2 "" H 2800 2300 50  0001 C CNN
@@
 	7400 2200 7400 2300
 $Comp
-L power:GND #PWR012
+L power:GND #PWR013
 U 1 1 5FB15A4D
 P 7400 2300
-F 0 "#PWR012" H 7400 2050 50  0001 C CNN
+F 0 "#PWR013" H 7400 2050 50  0001 C CNN
 F 1 "GND" H 7405 2127 50  0000 C CNN
 F 2 "" H 7400 2300 50  0001 C CNN
@@
 	7250 2100 7250 5250
 Wire Wire Line
-	7250 5250 2100 5250
-Wire Wire Line
-	2100 5250 2100 4500
-Wire Wire Line
-	2100 4500 2200 4500
+	7250 5250 1600 5250
+Wire Wire Line
+	1600 5250 1600 4500
+Wire Wire Line
+	1600 4500 1700 4500
 $Comp
 L power:PWR_FLAG #FLG01
@@
 Connection ~ 3500 4750
 $Comp
-L Device:R R1
+L Device:R R3
 U 1 1 5FB28AA5
 P 5000 1750
-F 0 "R1" H 5070 1796 50  0000 L CNN
+F 0 "R3" H 5070 1796 50  0000 L CNN
 F 1 "82k" H 5070 1705 50  0000 L CNN
 F 2 "Resistor_SMD:R_0603_1608Metric" V 4930 1750 50  0001 C CNN
@@
 $EndComp
 $Comp
-L Device:R R2
+L Device:R R4
 U 1 1 5FB2D53E
 P 5000 3650
-F 0 "R2" H 5070 3696 50  0000 L CNN
-F 1 "20k" H 5070 3605 50  0000 L CNN
+F 0 "R4" H 5070 3696 50  0000 L CNN
+F 1 "24k" H 5070 3605 50  0000 L CNN
 F 2 "Resistor_SMD:R_0603_1608Metric" V 4930 3650 50  0001 C CNN
 F 3 "~" H 5000 3650 50  0001 C CNN
@@
 $EndComp
 Wire Wire Line
-	2200 4300 2000 4300
-Wire Wire Line
-	2000 4300 2000 3400
-Wire Wire Line
-	2000 3400 5000 3400
-Wire Wire Line
-	5000 3400 5000 3500
-Wire Wire Line
-	5000 3400 5000 2200
-Connection ~ 5000 3400
+	1700 4300 1500 4300
+Wire Wire Line
+	1500 4300 1500 3400
+Wire Wire Line
+	1500 3400 5000 3400
 Wire Wire Line
 	4800 2200 5000 2200
@@
 	1    0    0    -1
 $EndComp
-Text Label 2050 3400 0    50   ~ 0
+Text Label 1550 3400 0    50   ~ 0
 ~ERR
 Text Label 5450 2000 0    50   ~ 0
@@
 PWM
 $Comp
-L Device:R R5
+L Device:R R7
 U 1 1 5FBD72C9
 P 6850 2300
-F 0 "R5" H 6920 2346 50  0000 L CNN
+F 0 "R7" H 6920 2346 50  0000 L CNN
 F 1 "24k" H 6920 2255 50  0000 L CNN
 F 2 "Resistor_SMD:R_0603_1608Metric" V 6780 2300 50  0001 C CNN
@@
 	6850 2450 6850 2550
 $Comp
-L power:GND #PWR013
+L power:GND #PWR012
 U 1 1 5FBDA3C1
 P 6850 2550
-F 0 "#PWR013" H 6850 2300 50  0001 C CNN
+F 0 "#PWR012" H 6850 2300 50  0001 C CNN
 F 1 "GND" H 6855 2377 50  0000 C CNN
 F 2 "" H 6850 2550 50  0001 C CNN
@@
 	1    0    0    1
 $EndComp
+Wire Wire Line
+	5000 2200 5000 3400
+$Comp
+L Device:R R1
+U 1 1 5FFE0D66
+P 2750 4050
+F 0 "R1" H 2820 4096 50  0000 L CNN
+F 1 "2k2" H 2820 4005 50  0000 L CNN
+F 2 "Resistor_SMD:R_0603_1608Metric" V 2680 4050 50  0001 C CNN
+F 3 "~" H 2750 4050 50  0001 C CNN
+F 4 "2.2kΩ 100mW 0603 resistor" H 2750 4050 50  0001 C CNN "Note"
+F 5 "MCWR06X2201FTL" H 2750 4050 50  0001 C CNN "Part Number"
+F 6 "Multicomp" H 2750 4050 50  0001 C CNN "Manufacturer"
+F 7 "0603" H 2750 4050 50  0001 C CNN "Package"
+F 8 "Farnell" H 2750 4050 50  0001 C CNN "Supplier"
+F 9 "2447320" H 2750 4050 50  0001 C CNN "Order Code"
+	1    2750 4050
+	1    0    0    -1
+$EndComp
+Wire Wire Line
+	2750 3900 2750 3800
+Connection ~ 2750 3800
+Wire Wire Line
+	2750 3800 3050 3800
+Wire Wire Line
+	3050 3900 3050 3800
+Connection ~ 3050 3800
+Wire Wire Line
+	3050 3800 3500 3800
+Wire Wire Line
+	3050 4200 3050 4400
+Connection ~ 3050 4400
+Wire Wire Line
+	2750 4200 2750 4300
+Connection ~ 2750 4300
+Wire Wire Line
+	2750 4300 3900 4300
+$Comp
+L Device:R R2
+U 1 1 5FFE7155
+P 3050 4050
+F 0 "R2" H 3120 4096 50  0000 L CNN
+F 1 "2k2" H 3120 4005 50  0000 L CNN
+F 2 "Resistor_SMD:R_0603_1608Metric" V 2980 4050 50  0001 C CNN
+F 3 "~" H 3050 4050 50  0001 C CNN
+F 4 "2.2kΩ 100mW 0603 resistor" H 3050 4050 50  0001 C CNN "Note"
+F 5 "MCWR06X2201FTL" H 3050 4050 50  0001 C CNN "Part Number"
+F 6 "Multicomp" H 3050 4050 50  0001 C CNN "Manufacturer"
+F 7 "0603" H 3050 4050 50  0001 C CNN "Package"
+F 8 "Farnell" H 3050 4050 50  0001 C CNN "Supplier"
+F 9 "2447320" H 3050 4050 50  0001 C CNN "Order Code"
+	1    3050 4050
+	1    0    0    -1
+$EndComp
+Connection ~ 5000 3400
+Wire Wire Line
+	5000 3400 5000 3500
 $EndSCHEMATC
